Commit message: update urdf lua and launch
for three lidat test with urdf

File: urdf/hokuyo_IMU.urdf (robot description, URDF)
Before this commit: robot cartographer_backpack_2d, 3 links, 2 joints
Joints:
- joint horizontal_laser_link_joint: origin xyz=0.1 0.2 1 -> xyz=-0.05 -0.15 0.7 rpy=0 0 3.14159265

File: urdf/three_hokuyo_ydy.urdf (robot description, URDF)
Before this commit: robot cartographer_backpack_2d, 4 links, 3 joints
Links:
- removed link vertical_laser_link
- added link vertical_left_laser_link; visual cylinder length=0.05 radius=0.03
- added link vertical_right_laser_link; visual cylinder length=0.05 radius=0.03
Joints:
- removed joint vertical_laser_link_joint
- added joint vertical_left_laser_link_joint: type fixed, parent base_link, child vertical_left_laser_link, origin xyz=0.1833109  0.2059131  0.2815776 rpy=-0.8259   1.4691    -0.7129
- added joint vertical_right_laser_link_joint: type fixed, parent base_link, child vertical_right_laser_link, origin xyz=0.0596314   0.0227044  0.4750975 rpy=-0.6614   1.4036    -2.0491
- joint horizontal_laser_link_joint: origin xyz=0.1007 0 0.0558 -> xyz=0.1475081  0.2252364  0.7851337 rpy=-0.0827   0.0731   0.1172
- joint imu_link_joint: origin xyz=0 0 0 rpy=0 0 0 -> xyz=0 0 0

File: urdf/three_hokuyo_ydy2.urdf (robot description, URDF)
Before this commit: robot cartographer_backpack_2d, 4 links, 3 joints
Links:
- removed link vertical_laser_link
- added link vertical_left_laser_link; visual cylinder length=0.05 radius=0.03
- added link vertical_right_laser_link; visual cylinder length=0.05 radius=0.03
Joints:
- removed joint vertical_laser_link_joint
- added joint vertical_left_laser_link_joint: type fixed, parent base_link, child vertical_left_laser_link, origin xyz=0.1309601  0.2834585  0.3186169 rpy=0.1315    -1.5430    -2.4868
- added joint vertical_right_laser_link_joint: type fixed, parent base_link, child vertical_right_laser_link, origin xyz=0.1446951   0.077  0.5380209 rpy=-0.7076   1.4941    -1.1402
- joint horizontal_laser_link_joint: origin xyz=0.1007 0 0.0558 -> xyz=0.1006602  0.1539847  0.8093709 rpy=-0.0068    -0.0030   0.0794
- joint imu_link_joint: origin xyz=0 0 0 rpy=0 0 0 -> xyz=0 0 0
