Commit message: add ..

File: urdf/trolley_2d.urdf (robot description, URDF)
Before this commit: robot cartographer_backpack_2d, 4 links, 3 joints
Links:
- removed link vertical_laser_link
- added link vertical_left_laser_link; visual cylinder length=0.05 radius=0.03
- added link vertical_right_laser_link; visual cylinder length=0.05 radius=0.03
Joints:
- removed joint vertical_laser_link_joint
- added joint vertical_left_laser_link_joint: type fixed, parent horizontal_laser_link, child vertical_left_laser_link, origin xyz=0.186045507305644 0.105986637974108 -1.33405283413285 rpy=-0.578851825592850 -1.54376984456986 -2.16548473925565
- added joint vertical_right_laser_link_joint: type fixed, parent horizontal_laser_link, child vertical_right_laser_link, origin xyz=0.184116048159474 -0.112894004828849 -0.952433033759406 rpy=-2.75577854779541 -1.51495918724335 -0.694204283574134
- joint horizontal_laser_link_joint: origin xyz=0.02 0.02 -0.035 -> xyz=0.0110 0 0.1810
- joint imu_link_joint: origin xyz=0 0 0 -> xyz=0 0 0 rpy=0.00932887273422234 -0.0245533259594644 1.56068650784503
